File: _pcb/_pcb_AUXsss/_AUX Mice Poke/mice poke simple v1.2.kicad_pcb (KiCad board)
At the start: 2 copper layers, 39 x 59.5 mm, 26 parts, among them IC1 SN74LVC1G125, Q1 BC817-40W, Q6 RTU002P02T106, U1 GP1A57HR_CUT2, X2 22-23-2041

Commit message: proceeding design VestibularVR H1
- Eagle version changed back to v.8.3.1
- proceeding design VestibularVR H1-module v1.0
- added Lick Sensor module v1.0
Parts:
- removed @HOLE0, @HOLE1, @HOLE2, @HOLE3, @HOLE4, @HOLE5: , 
- removed U$2: , mice poke simple v1.2:LOGO_7
- added J2: Conn_01x04, Connector_PinHeader_2.54mm:PinHeader_1x04_P2.54mm_Horizontal, F.Cu at (121.7, 98.1)
- DIO1: value (none) -> 22-23-2021
- J1: value (none) -> 215878-2
- LED1, LED2: value (none) -> LED3MM
Connections:
- net IR_IN renamed /IR_IN
- net LED renamed /LED
- J1 pad 8: (no net) -> unconnected-(J1-Pad8)
