File: _pcb/_pcb_AUXsss/_AUX Mice Poke/mice poke simple v1.2.kicad_sch (KiCad schematic)
At the start: 19 parts

Commit message: proceeding design VestibularVR H1
- Eagle version changed back to v.8.3.1
- proceeding design VestibularVR H1-module v1.0
- added Lick Sensor module v1.0
Parts:
- added J2: Conn_01x04, Connector_PinHeader_1.27mm:PinHeader_1x04_P1.27mm_Vertical, symbol Connector_Generic:Conn_01x04
- C1: value (none) -> 100nF; footprint (none) -> mice poke simple v1.2:C0402
- D1: value (none) -> NA; footprint (none) -> mice poke simple v1.2:SOD323-R
- DIO1, VALVE0: value (none) -> 22-23-2021; footprint (none) -> mice poke simple v1.2:22-23-2021
- IC1: value (none) -> SN74LVC1G125; footprint (none) -> mice poke simple v1.2:SOT23-5
- J1: value (none) -> 215878-2; footprint (none) -> mice poke simple v1.2:215878-2
- LED1, LED2: value (none) -> LED3MM; footprint (none) -> mice poke simple v1.2:LED3MM
- Q1: value (none) -> BC817-40W; footprint (none) -> mice poke simple v1.2:SOT323-BEC
- Q6: value (none) -> RTU002P02T106; footprint (none) -> mice poke simple v1.2:SOT323
- R1: value (none) -> 150; footprint (none) -> mice poke simple v1.2:R0402
- R2, R3: value (none) -> 300; footprint (none) -> mice poke simple v1.2:R0402
- R4: value (none) -> 3.3k; footprint (none) -> mice poke simple v1.2:R0402
- R5: value (none) -> 510; footprint (none) -> mice poke simple v1.2:R0402
- R6, R7: value (none) -> 10k; footprint (none) -> mice poke simple v1.2:R0402
- U1: value (none) -> GP1A57HR_CUT2; footprint (none) -> mice poke simple v1.2:GP1A57HR_CUT2
- X2: value (none) -> 22-23-2041; footprint (none) -> mice poke simple v1.2:22-23-2041
