File: _pcb/Harp Motor device H2-module v1.0/Harp Motor device H2-module v1.0.sch (EAGLE design)
At the start: 67 parts, among them IC1 FT232RL, IC2 74LVC1G07DBV, IC3 LP5907MFX-3.3, IC4 74LVC1G07DBV, IC5 74LVC1G07DBV, IC6 74LVC1G07DBV, IC7 USBLC6-2SC6, IC8 ATXMEGA32A4U, T1 DMG1012UW, T2 DMG1012UW, X1 2x5 header, X15 Main_plug, X2 2x5 header, X3 USB_MINI_B

Commit message: BOMs & start Harp Motor device H2-module v1.0
. almost final BOMs versions for VestibularVR H1-module v1.0 & Lick Sensor module v1.0
. start of new project Harp Motor device H2-module v1.0
Parts:
- removed C14, C15, C16, C17: 100nF, rcl:C-EUC0402K
- removed CAM_TRIGGERS: 1x4 case, con-molex:22-23-2041
- removed D1: BAT54, diode:BAT54
- removed IC2, IC4, IC5, IC6: 74LVC1G07DBV, VestibularVR H1-module v1.0:74LVC1G07DBV
- removed R1, R5: 0R, rcl:R-US_R0402
- removed R2, R6: DNI, rcl:R-US_R0402
- removed R4, R7: 10k, rcl:R-US_R0402
- removed R8, R9: 1M, rcl:R-US_R0402
- removed T1, T2: DMG1012UW, VestibularVR H1-module v1.0:DMG1012UW-7
- removed X1, X2: 2x5 header, con-samtec:TSW-105-02-S-D
- LICK_0, LICK_1: value 2x3 case -> 1x3 case
- REWARD_VALVES: value 22-23-2041 -> 1x4 case; MF (none) -> -; MPN (none) -> 282834-4 Digikey A98335-ND
Connections:
- removed net LICK_PORT_1: IC6.A, LICK_0-2.S, R9.2
- removed net LICK_PORT_2: IC5.A, LICK_1-2.S, R8.2
- removed net N$14: C15.1, IC2.VCC, R5.2, R6.2
- removed net N$4: CAM_TRIGGERS-4.S, IC2.Y
- removed net N$5: C16.1, IC4.VCC, R1.2, R2.2
- removed net N$68: D1.A, REWARD_VALVES-1.S, T2.D
- removed net N$8: CAM_TRIGGERS-2.S, IC4.Y
- removed net U_CAM1_TRIGGER: IC4.A, IC8.PC0/OC0A/SDA
- removed net U_CAM2_TRIGGER: IC2.A, IC8.OC0A/PD0
- removed net U_LICK_PORT_1: IC6.Y, IC8.PA0/ADC0/AREF
- removed net U_LICK_PORT_2: IC5.Y, IC8.PA1/ADC1
- removed net U_OPTICAL_FLOW_1_CS: IC8.PC4/OC1A/!SS, X1-2.1
- removed net U_OPTICAL_FLOW_1_INT: IC8.PB0/ADC8/AREF, X1-6.1
- removed net U_OPTICAL_FLOW_1_MISO: IC8.PC6/MISO/RXD1, X1-5.1
- removed net U_OPTICAL_FLOW_1_MOSI: IC8.PC5/OC1B/MOSI/XCK1, X1-4.1
- removed net U_OPTICAL_FLOW_1_SCK: IC8.PC7/SCK/TXD1/CLKO/EVO, X1-3.1
- removed net U_OPTICAL_FLOW_2_CS: IC8.OC1A/!SS!/PD4, X2-2.1
- removed net U_OPTICAL_FLOW_2_INT: IC8.PB1/ADC9, X2-6.1
- removed net U_OPTICAL_FLOW_2_MISO: IC8.D-/RXD1/MISO/PD6, X2-5.1
- removed net U_OPTICAL_FLOW_2_MOSI: IC8.OCB1/XCK1/MOSI/PD5, X2-4.1
- removed net U_OPTICAL_FLOW_2_SCK: IC8.D+/TXD1/SCK/PD7, X2-3.1
- removed net U_REWARD_VALVE_1: IC8.PA6/ADC6/AC1-OUT, R4.2, T2.G
- removed net U_REWARD_VALVE_2: IC8.PA7/ADC7/AC0-OUT, R7.2, T1.G
- net +12V: no longer D1.C, REWARD_VALVES-2.S, REWARD_VALVES-4.S
- net +3V3: no longer C14.1, C17.1, IC5.VCC, IC6.VCC, R1.1, R5.1, X1-1.1, X2-1.1
- net +3V3_U: now also SV2.2; no longer SV2.6
- net +5V: no longer R2.1, R6.1
- net GND: now also SV2.6; no longer C14.2, C15.2, C16.2, C17.2, CAM_TRIGGERS-1.S, CAM_TRIGGERS-3.S, IC2.GND, IC4.GND, IC5.GND, IC6.GND, R4.1, R7.1, R8.1, R9.1, SV2.2, T1.S, T2.S, X1-10.1, X1-7.1, X2-10.1, X2-7.1
- net HARP_H1_BOARD_RX: no longer IC8.OC0C/RXD0/PD2
- net HARP_H1_BOARD_TX: no longer IC8.OC0D/TXD0/PD3
- net HARP_H1_CLOCK_IN: no longer IC8.PC2/OC0C/RXD0
- net N$6: no longer REWARD_VALVES-3.S, T1.D
- net PDI_CLK: now also SV2.5; no longer SV2.1
- net PDI_DATA: now also SV2.1; no longer SV2.5
- net USBDM: now also C4.1, IC7.IO2@0; no longer C6.1, IC7.IO1@0
- net USBDP: now also C6.1, IC7.IO1@0; no longer C4.1, IC7.IO2@0
Other:
- note removed: "Camera_trigger 1 & 2"
- note removed: "Cammera Triggers"
- note removed: "DMG1012UW"
- note removed: "Lick Ports"
- note removed: "Lick port de OC maior R PDown ~50k"
- note removed: "Optical Flows"
- note removed: "PAA5100JE Optical tracking - can be powered @ 3V3 or 5V - line outputs level will depend of power"
- note removed: "Reward Valves"
- note removed: "lick sensor @3V3 GP1A57HRJ00F photointerrupter - design from FED3"
- note removed: "lick_port_1"
- note removed: "lick_port_2"
- note removed: "reward_valve_1"
- note removed: "reward_valve_2"
- moved on the sheet: C4, C6, D4, SV2
