File: _pcb/Harp Motor device H2-module v1.0/Harp Motor H2-module v1.0.sch (EAGLE design)
At the start: 53 parts, among them IC1 FT232RL, IC3 LP5907MFX-3.3, IC7 USBLC6-2SC6, IC8 ATXMEGA32A4U, J1 BNCPTH, J2 BNCPTH, J3 POWER_JACK, X1 22-23-2051, X15 Main_plug, X2 22-23-2051, X3 USB_MINI_B, X4 1x4 case, X5 1x3 case, X6 CLCK_JACK, X7 1x4 case, X8 22-23-2021

Commit message: VestibularVR H1BOM updates & Lick Sensor step on
- VestibularVR H1
. component ref updated
. BOM file updated

- Lick Sensor module v1.0
. still only on schematic design
Parts:
- removed J1, J2: BNCPTH, SparkFun-Connectors:BNCPTH
- removed J3: POWER_JACK, SparkFun-Connectors:POWER_JACK
- removed LICK_2, X5: 1x3 case, con-molex:22-23-2031
- removed X15: Main_plug, con-weidmueller-sl35:90G-5
- removed X8: 22-23-2021, con-molex:22-23-2021
- added C1, C14, C15, C16, C17: 100nF, rcl:C-EUC0402K
- added C23, C24: 4.7uF, rcl:C-EUC0603
- added CLKIN: CLCK_JACK, harp input expander:STEREO_JACK
- added HARP: Harp_Intrfc, con-weidmueller-sl35:90G-5
- added IC2, IC4, IC5: 74VHC1GT126DT1G, VestibularVR H1-module v1.0:74LVC1G07DBV
- added IC9: TLV70033DDCR, harp input expander:TLV700XX
- added R1: 330R, rcl:R-US_R0402
- added R11: DNI, rcl:R-US_R0402
- added R12, R13, R2, R4, R6, R7, R8: 10k, rcl:R-US_R0402
- added R5: 10R, rcl:R-US_R0402
- added R9: 1M, rcl:R-US_R0402
- added T1, T2, T3: DMG1012UW??, VestibularVR H1-module v1.0:DMG1012UW-7
- R10: value 330R -> 0R; device rcl:R-EU_R0402 -> rcl:R-US_R0402; MPN RC0402FR-07330RL -> RC0402JR-070RL; OEPS OEPS020037 -> OEPS020001
- R18, R34: DIGIKEY_PN 541-3959-1-ND -> 541-10.0KLDKR-ND
- X1: value 22-23-2051 -> USB_MINI_B; device con-molex:22-23-2051 -> VestibularVR H1-module v1.0:USB_MINI_B; MPN (none) -> UX60-MB-5S8; OEPS (none) -> OEPS070021
- X2: value 22-23-2051 -> Rot_Encoder
- X3: value USB_MINI_B -> EMRG_BUTT_IN_NO; device VestibularVR H1-module v1.0:USB_MINI_B -> con-molex:22-23-2021; MPN UX60-MB-5S8 -> (none); OEPS OEPS070021 -> (none)
- X4: value 1x4 case -> Hall_Effect; device con-molex:22-23-2041 -> con-molex:22-23-2031; MPN 282834-4 Digikey A98335-ND -> 282834-3; OEPS OEPS07 xxx1 -> OEPS070035
- X6: value CLCK_JACK -> BNCPTH; device harp input expander:STEREO_JACK -> SparkFun-Connectors:BNCPTH; MPN 35RASMT2BHNTRX -> (none); NOTES - -> (none); TYPE SMD -> (none)
- X7: value 1x4 case -> STEP_MOTOR; device con-molex:22-23-2041 -> con-molex:22-23-2051; MF - -> (none); MPN 282834-4 Digikey A98335-ND -> (none); OEPS OEPS07 xxx1 -> (none)
Connections:
- removed net N$4: LICK_2-3.S, X1-5.S, X2-5.S, X4-4.S
- new net A_PHASE: IC4.A, X2-3.S
- new net B_PHASE: IC5.A, X2-4.S
- new net CLOCK_IN: CLKIN.4, IC8.PB1/ADC9, R2.1
- new net EMERGENCY_INPUT: IC8.PB0/ADC8/AREF, R8.1, X3-1.S
- new net HALL_EFFCT_IN: IC2.A, X4-2.S
- new net LICK_PORT_1: R9.2
- new net N$103: CLKIN.1, R2.2, R5.2
- new net N$104: C24.1, IC9.OUT, R5.1
- new net N$5: C1.1, IC2.VCC, R10.2, R11.2, X4-3.S
- new net STEP_DIRECTION: T1.D, X7-3.S
- new net STEP_ENABLE: T2.D, X7-4.S
- new net STEP_PULSE: T3.D, X7-2.S
- new net U_A_PHASE: IC4.Y, IC8.PC4/OC1A/!SS
- new net U_B_PHASE: IC5.Y, IC8.PC3/OC0D/TXD0
- new net U_HALL_EFFCT_IN: IC2.Y, IC8.PA0/ADC0/AREF
- new net U_STEP_DIRECTION: IC8.PC6/MISO/RXD1, R12.2, T1.G
- new net U_STEP_ENABLE: IC8.PC5/OC1B/MOSI/XCK1, R6.2, T2.G
- new net U_STEP_PULSE: IC8.PC7/SCK/TXD1/CLKO/EVO, R13.2, T3.G
- new net V+: R8.2
- net +12V: now also HARP.1; no longer X15.1
- net +3V3: now also R10.1; no longer X5-3.S
- net +5V: now also C14.1, C17.1, C23.1, IC4.VCC, IC5.VCC, IC9.EN, IC9.IN, R11.1, X2-1.S, X7-1.S
- net GND: now also C1.2, C14.2, C15.2, C16.2, C17.2, C23.2, C24.2, CLKIN.5, HARP.5, IC2.GND, IC4.GND, IC5.GND, IC9.GND, R1.1, R12.1, R13.1, R4.1, R6.1, R7.1, R9.1, T1.S, T2.S, T3.S, X1.5, X2-5.S, X3-2.S, X6.GND, X7-5.S; no longer LICK_2-1.S, R10.1, X1-1.S, X15.5, X2-1.S, X3.5, X5-1.S, X6.5
- net HARP_H1_CLOCK_IN: now also HARP.4; no longer X1-2.S
- net HARP_H1_RX: now also HARP.3; no longer X1-3.S
- net HARP_H1_TX: now also HARP.2; no longer X1-4.S
- net N$1: now also X1.P$2; no longer X3.P$2
- net N$15: now also X1.P$3; no longer X3.P$3
- net N$2: now also X1.2; no longer X3.2
- net N$3: now also X1.3; no longer X3.3
- net N$9: now also R1.2; no longer R10.2
- net USB_POWER: now also X1.1; no longer X3.1
Other:
- note added: "Emergency Button NO in"
- note added: "H1 Harp interface InOut"
- note added: "Hall Effect sensor in"
- note added: "harp Clock in"
- note added: "in Stage rotation signal BNC plug: (be sure about)"
- note added: "main USB"
- note added: "out step motor control"
- note removed: "5V~24V inputs (??)"
- note removed: "CHECK VOLTAGE LEVEL OUTPUT!!!"
- note removed: "InOut H1 Harp interface"
- note removed: "Main Plug"
- note removed: "in Clock input"
- note removed: "in Emergency Button"
- note removed: "in Hall Effect sensor"
- note removed: "in jumpers to setup/test open or closed loop control??"
- note removed: "in sphere rotation signal"
- note removed: "in stage rotation signal ?? 2 signals??"
- note removed: "level translatioon 5V -> 3V3"
- note removed: "level translatioon 5V~24V -> 3V3"
- note removed: "out step motor cotrol"
- note removed: "out step motor driver"
- note removed: "to u; PullDown"
