File: _pcb/VestibularVR H1-module v1.0 - Copy/COPY VestibularVR H1-module v1.0.sch (EAGLE design)
At the start: 69 parts, among them IC1 FT232RL, IC10 74LVC1G126DBV, IC2 74VHC1GT126DT1G, IC3 LP5907MFX-3.3, IC4 74VHC1GT126DT1G, IC5 74VHC1GT126DT1G, IC6 74LVC1G125DBV, IC7 USBLC6-2SC6, IC8 ATXMEGA32A4U, IC9 TLV70033DDCR, T1 DMG1012UW??, T2 DMG1012UW??, T3 DMG1012UW??, X1 USB_MINI_B, X2 Rot_Encoder, X3 EMRG_BUTT_IN_NO, X4 Hall_Effect, X6 BNCPTH, X7 STEP_MOTOR

Commit message: Harp Motor device H2-module v1.0 - Schematic step on
Harp Motor device H2-module v1.0 - Schematic step on
Parts:
- removed C1: 100nF, rcl:C-EUC0402K
- removed C23, C24: 4.7uF, rcl:C-EUC0603
- removed CLKIN: CLCK_JACK, harp input expander:STEREO_JACK
- removed H2_MAIN_PLUG: be sure about plug type, con-weidmueller-sl35:90G-5
- removed IC10: 74LVC1G126DBV, 74xx-little-de:74LVC1G126DBV
- removed IC9: TLV70033DDCR, harp input expander:TLV700XX
- removed PWR1: DC_JACK2.1MM, harp camera controller:DC_JACK2.1MM
- removed R12, R13: 10k, rcl:R-US_R0402
- removed T3: DMG1012UW??, VestibularVR H1-module v1.0:DMG1012UW-7
- removed X4: Hall_Effect, con-molex:22-23-2031
- removed X6: BNCPTH, SparkFun-Connectors:BNCPTH
- removed X7: STEP_MOTOR, con-molex:22-23-2051
- added C15, C16: 100nF, rcl:C-EUC0402K
- added CAM_TRIGGERS, REWARD_VALVES: 1x4 case, con-molex:22-23-2041
- added D1: BAT54, diode:BAT54
- added LICK_0, LICK_1: 1x3 case, con-molex:22-23-2031
- added R10: 330R, rcl:R-EU_R0402
- added R4, R7: 10k, rcl:R-US_R0402
- added R9: 1M, rcl:R-US_R0402
- added X15: Main_plug, con-weidmueller-sl35:90G-5
- IC6: value 74LVC1G125DBV -> 74VHC1GT126DT1G; device 74xx-little-de:74LVC1G125DBV -> VestibularVR H1-module v1.0:74LVC1G07DBV; MPN (none) -> M74VHC1GT126DT1G; OEPS (none) -> OEPS080017
- R1: value 330R -> 0R; DIGIKEY_PN 541-10.0KLDKR-ND -> (none); MPN RC0402FR-07330RL -> RC0402JR-070RL; OEPS OEPS020037 -> OEPS020001
- R2, R6: value 10k -> DNI; DIGIKEY_PN 541-10.0KLDKR-ND -> (none); MPN CRCW040210K0FKED -> DNI; OEPS OEPS020030 -> DNI
- R5: value 10R -> 0R; DIGIKEY_PN qwee -> (none); MPN as -> RC0402JR-070RL; OEPS xx -> OEPS020001
- R8: value 10k -> 1M; DIGIKEY_PN 541-10.0KLDKR-ND -> 541-1.00MLCT-ND; MPN CRCW040210K0FKED -> CRCW04021M00FKED; OEPS OEPS020030 -> OEPS020026
- T1, T2: value DMG1012UW?? -> DMG1012UW; OEPS ?? escolhido muito power?? -> OEPS060010
- X1: value USB_MINI_B -> 2x5 header; device VestibularVR H1-module v1.0:USB_MINI_B -> con-samtec:TSW-105-02-S-D; MPN UX60-MB-5S8 -> 2x5 header; OEPS OEPS070021 -> n.a.
- X2: value Rot_Encoder -> 2x5 header; device con-molex:22-23-2051 -> con-samtec:TSW-105-02-S-D; MPN (none) -> 2x5 header; OEPS (none) -> n.a.
- X3: value EMRG_BUTT_IN_NO -> USB_MINI_B; device con-molex:22-23-2021 -> VestibularVR H1-module v1.0:USB_MINI_B; MPN (none) -> UX60-MB-5S8; OEPS (none) -> OEPS070021
Connections:
- removed net CLOCK_IN: CLKIN.4, IC8.PB1/ADC9, R2.1
- removed net EMERGENCY_INPUT: IC8.PB0/ADC8/AREF, R8.1, X3-1.S
- removed net ENCODER_A_PHASE: IC4.A, X2-3.S
- removed net ENCODER_B_PHASE: IC5.A, X2-4.S
- removed net HALL_EFFCT_IN: IC2.A, X4-1.S
- removed net HARP_H2_CLOCK_IN: H2_MAIN_PLUG.4, IC8.D-/RXD1/MISO/PD6
- removed net HARP_H2_RX: H2_MAIN_PLUG.3, IC8.OCB1/XCK1/MOSI/PD5
- removed net HARP_H2_TX: H2_MAIN_PLUG.2, IC8.OC1A/!SS!/PD4
- removed net N$103: CLKIN.1, R2.2, R5.2
- removed net N$104: C24.1, IC9.OUT, R5.1
- removed net STEP_DIRECTION: T1.D, X7-3.S
- removed net STEP_ENABLE: T2.D, X7-4.S
- removed net STEP_PULSE: T3.D, X7-2.S
- removed net U_ENCODER_A_PHASE: IC4.Y, IC8.PC4/OC1A/!SS
- removed net U_ENCODER_B_PHASE: IC5.Y, IC8.PC3/OC0D/TXD0
- removed net U_HALL_EFFCT_IN: IC2.Y, IC8.PA0/ADC0/AREF
- removed net U_STEP_DIRECTION: IC8.PC6/MISO/RXD1, R12.2, T1.G
- removed net U_STEP_ENABLE: IC8.PC5/OC1B/MOSI/XCK1, R6.2, T2.G
- removed net U_STEP_PULSE: IC8.PC7/SCK/TXD1/CLKO/EVO, R13.2, T3.G
- removed net V+: R8.2
- removed net VDD: H2_MAIN_PLUG.1, PWR1.1
- new net +12V: D1.C, D4.C, REWARD_VALVES-2.S, REWARD_VALVES-4.S, X15.1
- new net HARP_H1_BOARD_RX: IC8.OC0C/RXD0/PD2, X15.3
- new net HARP_H1_BOARD_TX: IC8.OC0D/TXD0/PD3, X15.2
- new net HARP_H1_CLOCK_IN: IC8.PC2/OC0C/RXD0, X15.4
- new net LICK_PORT_1: IC6.A, LICK_0-2.S, R9.2
- new net LICK_PORT_2: IC5.A, LICK_1-2.S, R8.2
- new net N$14: C15.1, IC2.VCC, R5.2, R6.2
- new net N$5: C16.1, IC4.VCC, R1.2, R2.2
- new net N$6: D4.A, REWARD_VALVES-3.S, T1.D
- new net N$68: D1.A, REWARD_VALVES-1.S, T2.D
- new net N$8: CAM_TRIGGERS-2.S, IC4.Y
- new net U_CAM1_TRIGGER: IC4.A, IC8.PC0/OC0A/SDA
- new net U_CAM2_TRIGGER: IC2.A, IC8.OC0A/PD0
- new net U_LICK_PORT_1: IC6.Y, IC8.PA0/ADC0/AREF
- new net U_LICK_PORT_2: IC5.Y, IC8.PA1/ADC1
- new net U_OPTICAL_FLOW_1_CS: IC8.PC4/OC1A/!SS, X1-2.1
- new net U_OPTICAL_FLOW_1_INT: IC8.PB0/ADC8/AREF, X1-6.1
- new net U_OPTICAL_FLOW_1_MISO: IC8.PC6/MISO/RXD1, X1-5.1
- new net U_OPTICAL_FLOW_1_MOSI: IC8.PC5/OC1B/MOSI/XCK1, X1-4.1
- new net U_OPTICAL_FLOW_1_SCK: IC8.PC7/SCK/TXD1/CLKO/EVO, X1-3.1
- new net U_OPTICAL_FLOW_2_CS: IC8.OC1A/!SS!/PD4, X2-2.1
- new net U_OPTICAL_FLOW_2_INT: IC8.PB1/ADC9, X2-6.1
- new net U_OPTICAL_FLOW_2_MISO: IC8.D-/RXD1/MISO/PD6, X2-5.1
- new net U_OPTICAL_FLOW_2_MOSI: IC8.OCB1/XCK1/MOSI/PD5, X2-4.1
- new net U_OPTICAL_FLOW_2_SCK: IC8.D+/TXD1/SCK/PD7, X2-3.1
- new net U_REWARD_VALVE_1: IC8.PA6/ADC6/AC1-OUT, R4.2, T2.G
- new net U_REWARD_VALVE_2: IC8.PA7/ADC7/AC0-OUT, R7.2, T1.G
- net +3V3: now also C14.1, C17.1, IC5.VCC, IC6.VCC, LICK_0-3.S, LICK_1-3.S, R1.1, R5.1, X1-1.1, X2-1.1; no longer C1.1, IC2.VCC, X4-2.S
- net +3V3_U: now also SV2.6; no longer SV2.2
- net +5V: now also R2.1, R6.1; no longer C14.1, C17.1, C23.1, IC4.VCC, IC5.VCC, IC9.EN, IC9.IN, X2-1.S
- net GND: now also C15.2, C16.2, CAM_TRIGGERS-1.S, CAM_TRIGGERS-3.S, IC6.GND, LICK_0-1.S, LICK_1-1.S, R10.1, R4.1, R7.1, R8.1, R9.1, SV2.2, X1-10.1, X1-7.1, X15.5, X2-10.1, X2-7.1, X3.5; no longer C1.2, C23.2, C24.2, CLKIN.5, H2_MAIN_PLUG.5, IC9.GND, PWR1.2, PWR1.3, R1.1, R12.1, R13.1, R6.1, SV2.6, T3.S, X1.5, X2-5.S, X3-2.S, X4-3.S, X7-5.S
- net N$1: now also X3.P$2; no longer X1.P$2
- net N$15: now also X3.P$3; no longer X1.P$3
- net N$2: now also X3.2; no longer X1.2
- net N$3: now also X3.3; no longer X1.3
- net N$4: now also CAM_TRIGGERS-4.S, IC2.Y; no longer X7-1.S
- net N$9: now also R10.2; no longer R1.2
- net PDI_CLK: now also SV2.1; no longer SV2.5
- net PDI_DATA: now also SV2.5; no longer SV2.1
- net USBDM: now also C6.1, IC7.IO1@0; no longer C4.1, IC7.IO2@0
- net USBDP: now also C4.1, IC7.IO2@0; no longer C6.1, IC7.IO1@0
- net USB_POWER: now also X3.1; no longer X1.1
Other:
- note added: "-to review USBDP & USBDP pin switched!!!"
- note added: "-to review pinout upside-down!!!"
- note added: "Camera_trigger 1 & 2"
- note added: "Cammera Triggers"
- note added: "DMG1012UW"
- note added: "Lick Ports"
- note added: "Lick port de OC maior R PDown ~50k"
- note added: "Main Plug"
- note added: "Optical Flows"
- note added: "PAA5100JE Optical tracking - can be powered @ 3V3 or 5V - line outputs level will depend of power"
- note added: "Reward Valves"
- note added: "lick sensor @3V3 GP1A57HRJ00F photointerrupter - design from FED3"
- note added: "lick_port_1"
- note added: "lick_port_2"
- note added: "reward_valve_1"
- note added: "reward_valve_2"
- note removed: "BNCs output: connected to two Teensy DAC Stage rotation signal (be sure about)"
- note removed: "Camera Controller - Clock_IN: PC2 - interrupst (?): PC0 PD0 - analog IN: ?? - camera Strobes (Interrupts?): CAM0: PA0=Strobe & PA1=PullUp CAM1: PD6=PullUp & PD7=Strobe"
- note removed: "H2 Harp External Power Input - straight to H1 module"
- note removed: "H2 Harp main IO plug"
- note removed: "USB"
- note removed: "check ferrite case"
- note removed: "check pinout not as in abstarct draw"
- note removed: "connection to Rotary Joint = H1 module"
- note removed: "input Emergency Button NO"
- note removed: "input Hall Effect home sensor"
- note removed: "input harp Clock"
- note removed: "input missing?? Treadmill Motion?? what have to do about it?"
- note removed: "input rotary encoder"
- note removed: "open drain output!! R pull-up out"
- note removed: "output step motor control"
- note removed: "pinout order: same as sensor"
- note removed: "power rail: - Vcc to stepper drive controller optos - DM542 stepper drive controller Vcc: = 5V~24V >> output voltage here can be 5V - Imax = ???"
- note removed: "rail de 5V ???? saida para o micro!!!"
- note removed: "sensor: WINGONEER JT0701"
- note removed: "use the other buffer with EN pin?? that way both buffers can be used"
- moved on the sheet: C10, C11, C12, C13, C14, C17, C2, C25, C26, C27, C28, C29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
